File: PCB/esc/Inverter.kicad_pcb (KiCad board)
At the start: 2 copper layers, 71.9 x 99.1 mm, 82 parts, among them J1 Conn_01x02, J2 Conn_01x05_Pin, J3 Conn_01x05_Pin, Q1 STP110N8F6, Q2 STP110N8F6, Q3 STP110N8F6, Q4 STP110N8F6, Q5 STP110N8F6, Q6 STP110N8F6, U1 XL7015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

Commit message: ported the code to STM32
Other:
- board text removed: "github.com/techn0man1ac/SimpleBLDC"
